File: Kicad/Oric.kicad_pcb (KiCad board)
At the start: 2 copper layers, 206.2 x 138.1 mm, 133 parts, among them IC1 LM7805, IC10 AY-3-8910, IC11 74LS00, IC2 LM386, IC20 74LS257, IC21 74LS04, IC22 74LS365, IC23 AD724, IC3 LM358, IC30 4464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

Commit message: Remix v1.2
Parts:
- G2: footprint Oric:tangerineleafpot -> Oric:tangerineleafpot_growth1
Connections:
- IC11 pad 1: ~{ROMDIS} -> ROMSEL
- IC11 pad 5: Net-(IC11-Pad3) -> ~{ROMDIS}
Routing:
- net ~{ROMDIS}: track 129.6 -> 117.1 mm
- net Net-(IC11-Pad3): track 5.08 -> 2.54 mm
- net ROMSEL: track 106.3 -> 108.9 mm
Other:
- board text added: "Thanks to: Lee (@morefunmakingit) Marko Šolajić (@msolajic) Simon Luce"
- board text added: "The Board Folk Team 2026"
- board text added: "v1.2 04/2026"
- board text removed: "Thanks to: Lee (@morefunmakingit) Marko Šolajić (@msolajic)"
- board text removed: "The Board Folk Team 2025"
- board text removed: "v1.1 01/2025"
