File: Kicad/oric_io.kicad_sch (KiCad schematic)
At the start: 68 parts, among them IC10 AY-3-8910, IC2 LM386, IC3 LM358, IC4 AY-3-8912, IC6 6522A

Commit message: Remix v1.2
Parts:
- TR1, TR2, TR3: symbol Device:Q_NPN_CBE -> Transistor_BJT:Q_NPN_CBE
